File: MovuinoBaseShield.kicad_sch (KiCad schematic)
At the start: 2 parts, among them J1 DF12-36NOLEGS-FEMALE, J3 DF12-36NOLEGS-MALE

Commit message: clean + comment
Parts:
- renumbered J3 to BOTTOM_DF12, J1 to TOP_DF12
Connections:
- net VCC is gone; now on net +3.3V: BOTTOM_DF12.32, TOP_DF12.31
- net IO36: now reaches BOTTOM_DF12.1
- net IO36: now also TOP_DF12.2
- net PB: now reaches BOTTOM_DF12.10
- net PB: now also TOP_DF12.9
- net IO35: now reaches BOTTOM_DF12.11
- net IO35: now also TOP_DF12.12
- net RESET: now reaches BOTTOM_DF12.12
- net RESET: now also TOP_DF12.11
- net IO32: now reaches BOTTOM_DF12.13
- net IO32: now also TOP_DF12.14
- net GPIO0: now reaches BOTTOM_DF12.14
- net GPIO0: now also TOP_DF12.13
- net IO33: now reaches BOTTOM_DF12.15
- net IO33: now also TOP_DF12.16
- net RXD: now reaches BOTTOM_DF12.16
- net RXD: now also TOP_DF12.15
- net IO25: now reaches BOTTOM_DF12.17
- net IO25: now also TOP_DF12.18
- net TXD: now reaches BOTTOM_DF12.18
- net TXD: now also TOP_DF12.17
- net IO26: now reaches BOTTOM_DF12.19
- net IO26: now also TOP_DF12.20
- net +5V: now reaches BOTTOM_DF12.2
- net +5V: now also BOTTOM_DF12.4, TOP_DF12.1, TOP_DF12.3
- net SCK: now reaches BOTTOM_DF12.20
- net SCK: now also TOP_DF12.19
- net IO27: now reaches BOTTOM_DF12.21
- net IO27: now also TOP_DF12.22
- net MOSI: now reaches BOTTOM_DF12.22
- net MOSI: now also TOP_DF12.21
- net IO14: now reaches BOTTOM_DF12.23
- net IO14: now also TOP_DF12.24
- net MISO: now reaches BOTTOM_DF12.24
- net MISO: now also TOP_DF12.23
- net IO15: now reaches BOTTOM_DF12.25
- net IO15: now also TOP_DF12.26
- net SDA: now reaches BOTTOM_DF12.26
- net SDA: now also TOP_DF12.25
- net IO12: now reaches BOTTOM_DF12.27
- net IO12: now also TOP_DF12.28
- net SCL: now reaches BOTTOM_DF12.28
- net SCL: now also TOP_DF12.27
- net IO13: now reaches BOTTOM_DF12.29
- net IO13: now also TOP_DF12.30
- net +3.3V: now reaches BOTTOM_DF12.30
- net +3.3V: now also TOP_DF12.29
- net IO4: now reaches BOTTOM_DF12.31
- net IO4: now also TOP_DF12.32
- net IO5: now reaches BOTTOM_DF12.33
- net IO5: now also TOP_DF12.34
- net GPIO2: now reaches BOTTOM_DF12.35
- net GPIO2: now also TOP_DF12.36
- net IO39: now reaches BOTTOM_DF12.5
- net IO39: now also TOP_DF12.6
- net BATT: now reaches BOTTOM_DF12.6
- net BATT: now also TOP_DF12.5
- net IO34: now reaches BOTTOM_DF12.7
- net IO34: now also TOP_DF12.8
- net VBATT: now reaches BOTTOM_DF12.8
- net VBATT: now also TOP_DF12.7
- net IO37: now reaches BOTTOM_DF12.9
- net IO37: now also TOP_DF12.10
- net ADC renamed IO38
Other:
- note added: "(A0 ADC1_CH0) BATT Monitoring"
- note added: "(TOUCH0 D9 ADC2_CH0) INT BUILTIN MPU"
- note added: "(TOUCH3 D6 ADC2_CH3) BUILTIN NEOPIXEL"
- note added: "(TOUCH4 D8 ADC2_CH4) PB_OUT"
- note added: "(TOUCH5 D7 ADC2_CH5) PS_HOLD"
- note added: "ADC1_CH1 A4"
- note added: "ADC1_CH2 A1"
- note added: "ADC1_CH3 A2"
- note added: "ADC1_CH4 A6 TOUCH9"
- note added: "ADC1_CH5 D1 TOUCH8"
- note added: "ADC1_CH6 A3"
- note added: "ADC1_CH7 A5"
- note added: "ADC2_CH2 X2 TOUCH2"
- note added: "ADC2_CH6 D5 TOUCH6"
- note added: "ADC2_CH7 D4 TOUCH7"
- note added: "ADC2_CH8 D2 DAC_1"
- note added: "ADC2_CH9 D3 DAC_2"
- note added: "GPIO5 X1"
- note added: "USE THIS CONNECTOR FOR BOTTOM SHIELD (PLUGGED UNDER MOVUINO)"
- note added: "USE THIS ONE FOR TOP SHIELD (PLUGGED ABOVE MOVUINO)"
- moved on the sheet: BOTTOM_DF12, TOP_DF12
